File: LEDDebug.kicad_sch (KiCad schematic)
At the start: 34 parts, among them J1 Conn_01x09_Pin

Commit message: Component sizing and placement update
Parts:
- removed GND1, GND2, GND3, GND4, GND5, GND6, GND7, GND8: TestPoint, TestPoint:TestPoint_THTPad_D1.5mm_Drill0.7mm, symbol Connector:TestPoint
- D1, D2, D3, D4, D5, D6, D7, D8: footprint LED_SMD:LED_0805_2012Metric_Pad1.15x1.40mm_HandSolder -> LED_SMD:LED_1206_3216Metric_Pad1.42x1.75mm_HandSolder
- R1, R2, R3, R4, R5, R6, R7, R8: footprint Resistor_SMD:R_0805_2012Metric_Pad1.20x1.40mm_HandSolder -> Resistor_SMD:R_1206_3216Metric_Pad1.30x1.75mm_HandSolder
- renumbered GND0 to GND1
Connections:
- net GND: now also R1.1, R2.1, R3.1, R4.1, R5.1, R6.1, R7.1, R8.1; no longer D1.1 (K), D2.1 (K), D3.1 (K), D4.1 (K), D5.1 (K), D6.1 (K), D7.1 (K), D8.1 (K)
- net TP1: now also D1.2 (A); no longer R1.2
- net TP2: now also D2.2 (A); no longer R2.2
- net TP3: now also D3.2 (A); no longer R3.2
- net TP4: now also D4.2 (A); no longer R4.2
- net TP5: now also D5.2 (A); no longer R5.2
- net TP6: now also D6.2 (A); no longer R6.2
- net TP7: now also D7.2 (A); no longer R7.2
- net TP8: now also D8.2 (A); no longer R8.2
- new net: D3.1 (K), R3.2
- new net: D7.1 (K), R7.2
- new net: D2.1 (K), R2.2
- new net: D4.1 (K), R4.2
- new net: D1.1 (K), R1.2
- new net: D6.1 (K), R6.2
- new net: D5.1 (K), R5.2
- new net: D8.1 (K), R8.2
Other:
- moved on the sheet: D1, R1
